File: hardware/sharkbait-tracker/rf_tx.kicad_sch (KiCad schematic)
At the start: 20 parts, among them J2 Conn_Coaxial_Small, U4 LLCC68, Y1 32MHz

Commit message: Combination antenna footprint and build automation
Parts:
- C11, C3, C5, C6: JLCPCB_CORRECTION 0;0;90 -> (none)
- J2: footprint Connector_Coaxial:SMA_Samtec_SMA-J-P-H-ST-EM1_EdgeMount -> Connector_Coaxial_Custom:SMA_Samtec_SMA-J-P-H-ST-EM1_EdgeMount_WireWhip; JLCPCB_IGNORE (none) -> ignore
- U4: footprint Package_DFN_QFN:QFN-24-1EP_4x4mm_P0.5mm_EP2.7x2.7mm -> Package_DFN_QFN:QFN-24-1EP_4x4mm_P0.5mm_EP2.7x2.7mm_ThermalVias; JLCPCB_CORRECTION (none) -> 0;0;-90; LCSC (none) -> C5120261
- Y1: LCSC (none) -> C843260
Changed lines of the file:
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@@
 			)
 		)
-		(property "JLCPCB_CORRECTION" "0;0;90"
+		(property "JLCPCB_CORRECTION" ""
 			(at 17.78 69.85 0)
 			(effects
@@
 			)
 		)
-		(property "JLCPCB_CORRECTION" "0;0;90"
+		(property "JLCPCB_CORRECTION" ""
 			(at 77.47 116.84 0)
 			(effects
@@
 			)
 		)
-		(property "Footprint" "Connector_Coaxial:SMA_Samtec_SMA-J-P-H-ST-EM1_EdgeMount"
+		(property "Footprint" "Connector_Coaxial_Custom:SMA_Samtec_SMA-J-P-H-ST-EM1_EdgeMount_WireWhip"
 			(at 231.14 93.98 0)
 			(effects
@@
 			)
 		)
+		(property "JLCPCB_IGNORE" "ignore"
+			(at 231.14 93.98 0)
+			(effects
+				(font
+					(size 1.27 1.27)
+				)
+				(hide yes)
+			)
+		)
 		(pin "1"
 		)
@@
 			)
 		)
-		(property "JLCPCB_CORRECTION" "0;0;90"
+		(property "JLCPCB_CORRECTION" ""
 			(at 30.48 69.85 0)
 			(effects
@@
 			)
 		)
+		(property "LCSC" "C843260"
+			(at 43.18 48.26 0)
+			(effects
+				(font
+					(size 1.27 1.27)
+				)
+				(hide yes)
+			)
+		)
 		(pin "2"
 		)
@@
 			)
 		)
-		(property "JLCPCB_CORRECTION" "0;0;90"
+		(property "JLCPCB_CORRECTION" ""
 			(at 85.09 68.58 0)
 			(effects
@@
 			)
 		)
-		(property "Footprint" "Package_DFN_QFN:QFN-24-1EP_4x4mm_P0.5mm_EP2.7x2.7mm"
+		(property "Footprint" "Package_DFN_QFN:QFN-24-1EP_4x4mm_P0.5mm_EP2.7x2.7mm_ThermalVias"
 			(at 57.15 74.93 0)
 			(effects
@@
 			(effects
 				(font
+					(size 1.27 1.27)
+				)
+				(hide yes)
+			)
+		)
+		(property "LCSC" "C5120261"
+			(at 57.15 96.52 0)
+			(effects
+				(font
+					(size 1.27 1.27)
+				)
+				(hide yes)
+			)
+		)
+		(property "JLCPCB_CORRECTION" "0;0;-90"
+			(at 57.15 96.52 0)
+			(effects
+				(font
